Commit message: Actuator command was updated
Signed-off-by: Juan S. Cely G. <juanscelyg@gmail.com>

File: robots/robot.urdf.xacro (robot description, xacro)
@@ -18,14 +18,14 @@
     <xacro:base prefix="$(arg prefix)"/>
     <!-- rotors -->
+    <xacro:rotor_ccw prefix="0" parent="base_link">
+        <origin xyz="${rotor_offset_x} ${rotor_offset_y} ${rotor_offset_z}" rpy="0 0 0"/>
+    </xacro:rotor_ccw>
     <xacro:rotor_cw prefix="1" parent="base_link">
-        <origin xyz="${rotor_offset_x} ${rotor_offset_y} ${rotor_offset_z}" rpy="0 0 0"/>
+        <origin xyz="${rotor_offset_x} -${rotor_offset_y} ${rotor_offset_z}" rpy="0 0 0"/>
     </xacro:rotor_cw>
-    <xacro:rotor_ccw prefix="2" parent="base_link">
-        <origin xyz="${rotor_offset_x} -${rotor_offset_y} ${rotor_offset_z}" rpy="0 0 0"/>
-    </xacro:rotor_ccw>
-    <xacro:rotor_cw prefix="3" parent="base_link">
+    <xacro:rotor_cw prefix="2" parent="base_link">
         <origin xyz="-${rotor_offset_x} ${rotor_offset_y} ${rotor_offset_z}" rpy="0 0 0"/>
     </xacro:rotor_cw>
-    <xacro:rotor_ccw prefix="4" parent="base_link">
+    <xacro:rotor_ccw prefix="3" parent="base_link">
         <origin xyz="-${rotor_offset_x} -${rotor_offset_y} ${rotor_offset_z}" rpy="0 0 0"/>
     </xacro:rotor_ccw>
@@ -37,3 +37,30 @@
         <origin xyz="0.0 0.0 0.0" rpy="0 0 0"/>
     </xacro:sensor_barometer>
+    <!-- Plugins -->
+    <plugin
+      filename="gz-sim-pose-publisher-system"
+      name="gz::sim::systems::PosePublisher">
+      <publish_link_pose>true</publish_link_pose>
+      <publish_model_pose>false</publish_model_pose>
+      <publish_sensor_pose>true</publish_sensor_pose>
+      <publish_visual_pose>false</publish_visual_pose>
+      <publish_nested_model_pose>true</publish_nested_model_pose>
+      <use_pose_vector_msg>true</use_pose_vector_msg>
+      <static_publisher>true</static_publisher>
+    </plugin>
+    <plugin filename="gz-sim-joint-state-publisher-system"
+        name="gz::sim::systems::JointStatePublisher">
+      <topic>joint_states</topic>
+      <joint>rotor_0_joint</joint>
+      <joint>rotor_1_joint</joint>
+      <joint>rotor_2_joint</joint>
+      <joint>rotor_3_joint</joint>
+    </plugin>
+        <plugin
+      filename="gz-sim-odometry-publisher-system"
+      name="gz::sim::systems::OdometryPublisher">
+      <dimensions>3</dimensions>
+      <odom_frame>odom</odom_frame>
+      <robot_base_frame>base_link</robot_base_frame>
+    </plugin>
 </robot>

File: urdf/base/base.urdf.xacro (robot description, xacro)
@@ -8,5 +8,5 @@
             <inertial>
                 <origin xyz="0 0 0" rpy="0 0 0"/>
-                <mass value="1.0"/>
+                <mass value="0.05"/>
                 <inertia  ixx="0.017" ixy="0.0"  ixz="0.0"  iyy="0.017"  iyz="0.0"  izz="0.034" />
             </inertial>

File: urdf/rotor/rotor.urdf.xacro (robot description, xacro)
@@ -9,5 +9,5 @@
         <child link="rotor_${prefix}_link"/>
         <axis xyz="0 0 1" rpy="0 0 0" />
-        <limit effort="5000" velocity="100"/>
+        <limit effort="5000" velocity="10000"/>
         <dynamics damping="0.05" friction="0.1"/>
     </joint>
@@ -15,5 +15,5 @@
         <inertial>
             <origin xyz="0 0 0" rpy="0 0 0"/>
-            <mass value="10.0"/>
+            <mass value="0.005"/>
             <inertia ixx="0.02975" ixy="0" ixz="0" iyy="0.03087" iyz="0" izz="0.00191"/>
         </inertial>
@@ -39,8 +39,8 @@
         <timeConstantUp>0.0125</timeConstantUp>
         <timeConstantDown>0.025</timeConstantDown>
-        <maxRotVelocity>1000.0</maxRotVelocity>
-        <motorConstant>8.54858e-06</motorConstant>
-        <momentConstant>0.016</momentConstant>
-        <commandSubTopic>command/motor_${prefix}_speed</commandSubTopic>
+        <maxRotVelocity>4760.0</maxRotVelocity>
+        <motorConstant>3.3e-08</motorConstant>
+        <momentConstant>0.0016</momentConstant>
+        <commandSubTopic>command/motor_speed</commandSubTopic>
         <actuator_number>${prefix}</actuator_number>
         <rotorDragCoefficient>8.06428e-05</rotorDragCoefficient>
@@ -58,5 +58,5 @@
         <child link="rotor_${prefix}_link"/>
         <axis xyz="0 0 1" rpy="0 0 0" />
-        <limit effort="5000" velocity="100"/>
+        <limit effort="5000" velocity="10000"/>
         <dynamics damping="0.05" friction="0.1"/>
     </joint>
@@ -64,5 +64,5 @@
         <inertial>
             <origin xyz="0 0 0" rpy="0 0 0"/>
-            <mass value="10.0"/>
+            <mass value="0.005"/>
             <inertia ixx="0.02975" ixy="0" ixz="0" iyy="0.03087" iyz="0" izz="0.00191"/>
         </inertial>
@@ -88,8 +88,8 @@
         <timeConstantUp>0.0125</timeConstantUp>
         <timeConstantDown>0.025</timeConstantDown>
-        <maxRotVelocity>1000.0</maxRotVelocity>
-        <motorConstant>8.54858e-06</motorConstant>
-        <momentConstant>0.016</momentConstant>
-        <commandSubTopic>command/motor_${prefix}_speed</commandSubTopic>
+        <maxRotVelocity>4760.0</maxRotVelocity>
+        <motorConstant>3.3e-08</motorConstant>
+        <momentConstant>0.0016</momentConstant>
+        <commandSubTopic>command/motor_speed</commandSubTopic>
         <actuator_number>${prefix}</actuator_number>
         <rotorDragCoefficient>8.06428e-05</rotorDragCoefficient>
